File: Keyhorde425/Keyhorde425.sch (KiCad schematic (older format))
At the start: 110 parts, among them J1 MX-NoLED, J2 USB_C_Receptacle_USB2.0, K1 MX-NoLED, M1 MX-NoLED, P1 MX-NoLED, Q1 MX-NoLED, SW1 SW_Push, T1 MX-NoLED, U1 ATmega32U4-AU, U2 MX-NoLED, X1 MX-NoLED, Y1 16MHz, Y2 MX-NoLED

Commit message: Updated schematic with bad diode footprint
Parts:
- removed Diode40: SOD-123, Diode_THT:D_5KP_P7.62mm_Vertical_AnodeUp, symbol Device:D_Small
- removed R-MOD-3: MX-NoLED, MX_Alps_Hybrid:MX-1U, symbol MX_Alps_Hybrid:MX-NoLED
- renumbered ,1 to ,, .1 to ., /1 to /, ;1 to ;, A1 to A, B1 to B, BKSP1 to BKSP, C8 to C, D1 to D, E1 to E, ENTR1 to ENTR, Esc1 to Esc, F1 to F, G1 to G, H1 to H, I1 to I, J1 to J, K1 to K, L1 to L, L-SHFT1 to L-SHFT, M1 to M, N1 to N, O1 to O, P1 to P, Q1 to Q, R5 to R, R-SHFT1 to R-SHFT, S1 to S, T1 to T, Tab1 to Tab, U2 to U, V1 to V, W1 to W, X1 to X, Y2 to Y, Z1 to Z
Connections:
- net COL10: now also R-MOD-1.1 (COL)
- net COL11: now also R-MOD-2.1 (COL)
- net COL4: no longer CTR-MOD1.1 (COL)
- net COL5: now also CTR-MOD1.1 (COL); no longer SPC-2.1 (COL)
- net COL6: no longer MOD-2.1 (COL)
- net COL7: now also SPC-2.1 (COL); no longer R-MOD-1.1 (COL)
- net COL8: no longer R-MOD-2.1 (COL)
- net COL9: now also MOD-2.1 (COL)
Other:
- moved on the sheet: CTR-MOD1, Diode20, Diode24, Diode28, Diode32, Diode36, MOD-2, R-MOD-1, R-MOD-2, SPC-2

Commit message: Add marbastlib submodule
Parts:
- Diode1, Diode10, Diode11, Diode12, Diode13, Diode14, Diode15, Diode16, Diode17, Diode18, Diode19, Diode2, Diode20, Diode21, Diode22, Diode23, Diode24, Diode25, Diode26, Diode27, Diode28, Diode29, Diode3, Diode30, Diode31, Diode32, Diode33, Diode34, Diode35, Diode36, Diode37, Diode38, Diode39, Diode4, Diode41, Diode42, Diode43, Diode44, Diode45, Diode46, Diode5, Diode6, Diode7, Diode8, Diode9: footprint Diode_THT:D_5KP_P7.62mm_Vertical_AnodeUp -> Diode_SMD:D_SOD-123
- renumbered , to ,-key, . to .-key, / to /-key, ; to ;-key, A to A-key, B to B-key, BKSP to BKSP-key, C to C-key, D to D-key, E to E-key, ENTR to ENTR-key, Esc to Esc-key, F to F-key, G to G-key, H to H-key, I to I-key, J to J-key, K to K-key, L-SHFT to L-SHFT-key, L to L-key, M to M-key, N to N-key, O to O-key, P to P-key, Q to Q-key, R-SHFT to R-SHFT-key, R to R-key, S to S-key, T to T-key, Tab to Tab-key, U to U-key, V to V-key, W to Wkey, X to X-key, Y to Y-key, Z to Z-key

Commit message: Halfway done routing traces (hopefully)
Layout finished barring reset switch, a better Type-C port, and any issues. Begun routing.
Parts:
- ,-key1: renamed from ,-key; footprint MX_Alps_Hybrid:MX-1U -> MX_Alps_Hybrid:MX-1U-NoLED
- .-key1: renamed from .-key; footprint MX_Alps_Hybrid:MX-1U -> MX_Alps_Hybrid:MX-1U-NoLED
- /-key1: renamed from /-key; footprint MX_Alps_Hybrid:MX-1U -> MX_Alps_Hybrid:MX-1U-NoLED
- ;-key1: renamed from ;-key; footprint MX_Alps_Hybrid:MX-1U -> MX_Alps_Hybrid:MX-1U-NoLED
- A-key1: renamed from A-key; footprint MX_Alps_Hybrid:MX-1U -> MX_Alps_Hybrid:MX-1U-NoLED
- B-key1: renamed from B-key; footprint MX_Alps_Hybrid:MX-1U -> MX_Alps_Hybrid:MX-1U-NoLED
- BKSP-key1: renamed from BKSP-key; footprint MX_Alps_Hybrid:MX-1U -> MX_Alps_Hybrid:MX-1.75U-NoLED
- C-key1: renamed from C-key; footprint MX_Alps_Hybrid:MX-1U -> MX_Alps_Hybrid:MX-1U-NoLED
- CTR-MOD-1: renamed from CTR-MOD1; footprint MX_Alps_Hybrid:MX-1U -> MX_Alps_Hybrid:MX-1.25U-NoLED
- D-key1: renamed from D-key; footprint MX_Alps_Hybrid:MX-1U -> MX_Alps_Hybrid:MX-1U-NoLED
- E-key1: renamed from E-key; footprint MX_Alps_Hybrid:MX-1U -> MX_Alps_Hybrid:MX-1U-NoLED
- ENTR-key1: renamed from ENTR-key; footprint MX_Alps_Hybrid:MX-1U -> MX_Alps_Hybrid:MX-1.5U-NoLED
- Esc-key1: renamed from Esc-key; footprint MX_Alps_Hybrid:MX-1U -> MX_Alps_Hybrid:MX-1U-NoLED
- F-key1: renamed from F-key; footprint MX_Alps_Hybrid:MX-1U -> MX_Alps_Hybrid:MX-1U-NoLED
- G-key1: renamed from G-key; footprint MX_Alps_Hybrid:MX-1U -> MX_Alps_Hybrid:MX-1U-NoLED
- H-key1: renamed from H-key; footprint MX_Alps_Hybrid:MX-1U -> MX_Alps_Hybrid:MX-1U-NoLED
- I-key1: renamed from I-key; footprint MX_Alps_Hybrid:MX-1U -> MX_Alps_Hybrid:MX-1U-NoLED
- J-key1: renamed from J-key; footprint MX_Alps_Hybrid:MX-1U -> MX_Alps_Hybrid:MX-1U-NoLED
- K-key1: renamed from K-key; footprint MX_Alps_Hybrid:MX-1U -> MX_Alps_Hybrid:MX-1U-NoLED
- L-MOD-1, L-MOD-3: footprint MX_Alps_Hybrid:MX-1U -> MX_Alps_Hybrid:MX-1U-NoLED
- L-MOD-2: footprint MX_Alps_Hybrid:MX-1U -> MX_Alps_Hybrid:MX-1.25U
- L-SHFT-key1: renamed from L-SHFT-key; footprint MX_Alps_Hybrid:MX-1U -> MX_Alps_Hybrid:MX-1.75U-NoLED
- L-key1: renamed from L-key; footprint MX_Alps_Hybrid:MX-1U -> MX_Alps_Hybrid:MX-1U-NoLED
- M-key1: renamed from M-key; footprint MX_Alps_Hybrid:MX-1U -> MX_Alps_Hybrid:MX-1U-NoLED
- N-key1: renamed from N-key; footprint MX_Alps_Hybrid:MX-1U -> MX_Alps_Hybrid:MX-1U-NoLED
- O-key1: renamed from O-key; footprint MX_Alps_Hybrid:MX-1U -> MX_Alps_Hybrid:MX-1U-NoLED
- P-key1: renamed from P-key; footprint MX_Alps_Hybrid:MX-1U -> MX_Alps_Hybrid:MX-1U-NoLED
- Q-key1: renamed from Q-key; footprint MX_Alps_Hybrid:MX-1U -> MX_Alps_Hybrid:MX-1U-NoLED
- R-MOD-1: renamed from MOD-2; footprint MX_Alps_Hybrid:MX-1U -> MX_Alps_Hybrid:MX-1U-NoLED
- R-MOD-2: renamed from R-MOD-1; footprint MX_Alps_Hybrid:MX-1U -> MX_Alps_Hybrid:MX-1.25U
- R-MOD-3: renamed from R-MOD-2; footprint MX_Alps_Hybrid:MX-1U -> MX_Alps_Hybrid:MX-1U-NoLED
- R-SHFT-key1: renamed from R-SHFT-key; footprint MX_Alps_Hybrid:MX-1U -> MX_Alps_Hybrid:MX-1U-NoLED
- R-key1: renamed from R-key; footprint MX_Alps_Hybrid:MX-1U -> MX_Alps_Hybrid:MX-1U-NoLED
- S-key1: renamed from S-key; footprint MX_Alps_Hybrid:MX-1U -> MX_Alps_Hybrid:MX-1U-NoLED
- SPC-1: footprint MX_Alps_Hybrid:MX-1U -> MX_Alps_Hybrid:MX-2.25U-NoLED
- SPC-2: footprint MX_Alps_Hybrid:MX-1U -> MX_Alps_Hybrid:MX-2.75U-NoLED
- T-key1: renamed from T-key; footprint MX_Alps_Hybrid:MX-1U -> MX_Alps_Hybrid:MX-1U-NoLED
- Tab-key1: renamed from Tab-key; footprint MX_Alps_Hybrid:MX-1U -> MX_Alps_Hybrid:MX-1.25U-NoLED
- U-key1: renamed from U-key; footprint MX_Alps_Hybrid:MX-1U -> MX_Alps_Hybrid:MX-1U-NoLED
- V-key1: renamed from V-key; footprint MX_Alps_Hybrid:MX-1U -> MX_Alps_Hybrid:MX-1U-NoLED
- Wkey1: renamed from Wkey; footprint MX_Alps_Hybrid:MX-1U -> MX_Alps_Hybrid:MX-1U-NoLED
- X-key1: renamed from X-key; footprint MX_Alps_Hybrid:MX-1U -> MX_Alps_Hybrid:MX-1U-NoLED
- Y-key1: renamed from Y-key; footprint MX_Alps_Hybrid:MX-1U -> MX_Alps_Hybrid:MX-1U-NoLED
- Z-key1: renamed from Z-key; footprint MX_Alps_Hybrid:MX-1U -> MX_Alps_Hybrid:MX-1U-NoLED
- renumbered Diode35 to ,-D, Diode39 to .-D, Diode43 to /-D, Diode42 to ;-D, Diode6 to A-D, R4 to ATGroundRes, C6 to ATucap, Diode23 to B-D, Diode44 to BKSP-D, Diode15 to C-D, Diode20 to CTR-MOD-D, Y1 to Cry, C2 to CryCap1, C3 to CryCap2, R2 to D+R, Diode14 to D-D, R1 to D-R, Diode13 to E-D, Diode45 to ENTR-D, Diode1 to ESC-D, Diode18 to F-D, Diode22 to G-D, Diode26 to H-D, Diode33 to I-D, Diode30 to J-D, Diode34 to K-D, Diode38 to L-D, Diode4 to L-MOD-1-D, Diode8 to L-MOD-2-D, Diode12 to L-MOD-3-D, Diode3 to L-SHFT-D, Diode31 to M-D, Diode27 to N-D, Diode37 to O-D, Diode41 to P-D, Diode5 to Q-D, Diode17 to R-D, Diode28 to R-MOD-1-D, Diode32 to R-MOD-2-D, Diode36 to R-MOD-3-D, Diode46 to R-SHFT-D, Diode10 to S-D, Diode16 to SPC-1-D, Diode24 to SPC-2-D, Diode21 to T-D, Diode2 to Tab-D, Diode29 to U-D, Diode19 to V-D, Diode9 to W-D, Diode11 to X-D, Diode25 to Y-D, Diode7 to Z-D

Commit message: Take two on routing
Wiped all routing and started over in preparation for wiping all routing and starting over again next time.
Parts:
- L-MOD-2, R-MOD-2: footprint MX_Alps_Hybrid:MX-1.25U -> MX_Alps_Hybrid:MX-1.25U-NoLED
- renumbered ,-D to ,-D1, .-D to .-D1, /-D to /-D1, ;-D to ;-D1, A-D to A-D1, ATGroundRes to ATGroundRes1, ATucap to ATucap1, B-D to B-D1, BKSP-D to BKSP-D1, C-D to C-D1, CTR-MOD-D to CTR-MOD-D1, Cry to Cry1, D+R to D+R1, D-D to D-D1, D-R to D-R1, E-D to E-D1, ENTR-D to ENTR-D1, ESC-D to ESC-D1, F-D to F-D1, G-D to G-D1, H-D to H-D1, I-D to I-D1, J-D to J-D1, K-D to K-D1, L-D to L-D1, L-MOD-1-D to L-MOD-1-D1, L-MOD-2-D to L-MOD-2-D1, L-MOD-3-D to L-MOD-3-D1, L-SHFT-D to L-SHFT-D1, M-D to M-D1, N-D to N-D1, O-D to O-D1, P-D to P-D1, Q-D to Q-D1, R-D to R-D1, R-MOD-1-D to R-MOD-1-D1, R-MOD-2-D to R-MOD-2-D1, R-MOD-3-D to R-MOD-3-D1, R-SHFT-D to R-SHFT-D1, S-D to S-D1, SPC-1-D to SPC-1-D1, SPC-2-D to SPC-2-D1, T-D to T-D1, Tab-D to Tab-D1, U-D to U-D1, V-D to V-D1, W-D to W-D1, X-D to X-D1, Y-D to Y-D1, Z-D to Z-D1
