File: Keyhorde425/Keyhorde425.kicad_pcb (KiCad board)
At the start: 2 copper layers, 247.7 x 80.9 mm, 108 parts, among them J2 USB_C_Receptacle_USB2.0, SW1 SW_Push, U1 ATmega32U4-AU, Y1 16MHz

Commit message: Take two on routing
Wiped all routing and started over in preparation for wiping all routing and starting over again next time.
Parts:
- removed R2: 22, Resistor_SMD:R_0805_2012Metric
- added D+R1: 22, Resistor_SMD:R_0805_2012Metric, F.Cu at (242.2, 102.8)
- ,-D1, .-D1, /-D1, ;-D1, A-D1, B-D1, BKSP-D1, C-D1, C1, C4, C5, C7, CTR-MOD-D1, D-D1, E-D1, ESC-D1, F-D1, Fuse1, G-D1, H-D1, I-D1, J-D1, J2, K-D1, L-D1, L-MOD-1-D1, L-MOD-2-D1, L-MOD-3-D1, L-SHFT-D1, M-D1, N-D1, O-D1, P-D1, Q-D1, R-D1, R-MOD-1-D1, R-MOD-2-D1, R-MOD-3-D1, R-SHFT-D1, R3, S-D1, SPC-1-D1, SPC-2-D1, T-D1, Tab-D1, U-D1, U1, USB2pull-down1, USB2pull-down2, V-D1, W-D1, X-D1, Y-D1, Z-D1: moved to F.Cu
- ATGroundRes1: renamed from R4; moved to F.Cu
- ATucap1: renamed from C6; moved to F.Cu
- Cry1: renamed from Y1; moved to F.Cu
- CryCap1: renamed from C2; moved to F.Cu
- CryCap2: renamed from C3; moved to F.Cu
- D-R1: renamed from R1; moved to F.Cu
- L-MOD-2, R-MOD-2: footprint MX_Alps_Hybrid:MX-1.25U -> MX_Alps_Hybrid:MX-1.25U-NoLED
- moved USB2pull-down1 104.4 mm to (244.6, 103.1)
- moved J2 99.7 mm to (241.2, 95.0), turned to 180 degrees
- moved D-R1 97.2 mm to (240.2, 102.8)
- moved USB2pull-down2 94.9 mm to (237.7, 103.1)
- moved SW1 25.8 mm to (266.7, 97.8)
- moved C7 23.7 mm to (242.1, 128.5), turned to 0 degrees
- moved C4 18.7 mm to (242.1, 126.6), turned to 0 degrees
- moved SPC-2-D1 18.6 mm to (189.7, 153.2), turned to 270 degrees
- moved CryCap1 17.5 mm to (232.0, 113.2), turned to 180 degrees
- moved R-MOD-3-D1 16.4 mm to (268.3, 153.2), turned to 270 degrees
- moved R-SHFT-D1 16.4 mm to (268.3, 134.1), turned to 270 degrees
- moved T-D1 16.4 mm to (139.7, 96.0), turned to 270 degrees
- moved P-D1 14.2 mm to (232.6, 96.0), turned to 270 degrees
- moved SPC-1-D1 14.2 mm to (118.3, 153.2), turned to 270 degrees
- moved ATucap1 13.7 mm to (242.1, 122.8), turned to 0 degrees
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Routing:
- net COL3: track 61.3 -> 254.1 mm
- net COL4: track 42.2 -> 220.3 mm
- net COL5: track 60.3 -> 210.2 mm
- net Net-(D+R1-Pad1): track 104.7 -> 10.6 mm, vias 0 -> 2
- net Net-(D-R1-Pad1): track 102.2 -> 8.64 mm, vias 3 -> 2
- net COL9: track 61.2 -> 118.8 mm
- net ROW1: track 220.7 -> 271.5 mm, vias 0 -> 12
- net GND: track 62.7 -> 39.2 mm, vias 2 -> 0
- net Net-(R3-Pad2): track 20.4 -> 0.00 mm, vias 2 -> 0
- net Net-(SPC-2-D1-Pad2): track 23.3 -> 4.73 mm
- net COL11: track 57.5 -> 41.1 mm, vias 0 -> 1
- net ROW0: track 280.5 -> 296.6 mm, vias 0 -> 13
- net +5V: track 21.7 -> 6.18 mm
- net ROW2: track 249.5 -> 264.8 mm, vias 2 -> 13
- net COL10: track 60.3 -> 74.4 mm
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
Commit message: First draft routing
First draft of the PCB with certifiably bad routing complete. Still needs better USB Type-C footprint/receptacle
Parts:
- moved R3 30.1 mm to (265.2, 104.6), turned to 90 degrees
- moved Fuse1 24.8 mm to (248.3, 95.6)
- moved ATGroundRes1 17.7 mm to (268.6, 104.6)
Routing:
- net COL0: track 65.2 -> 281.0 mm, vias 1 -> 2
- net COL1: track 68.3 -> 264.8 mm, vias 0 -> 2
- net COL2: track 67.5 -> 247.5 mm, vias 0 -> 2
- net +5V: track 6.18 -> 118.9 mm
- net COL6: track 44.0 -> 149.5 mm, vias 0 -> 2
- net COL7: track 62.1 -> 142.5 mm, vias 0 -> 2
- net COL10: track 74.4 -> 153.3 mm
- net GND: track 39.2 -> 114.3 mm, vias 0 -> 2
- net COL9: track 118.8 -> 185.0 mm
- net COL8: track 44.0 -> 101.2 mm, vias 0 -> 2
- net COL4: track 220.3 -> 273.6 mm
- net COL5: track 210.2 -> 262.4 mm
- net Net-(R3-Pad2): track 0.00 -> 48.9 mm, vias 0 -> 4
- net COL3: track 254.1 -> 300.9 mm
- net Net-(Cry1-Pad3): track 0.00 -> 35.8 mm, vias 0 -> 4
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